File: Constant register/Constant register.kicad_sch (KiCad schematic)
At the start: 30 parts, among them J1 Conn_01x16, J2 Conn_01x04, U1 74HCT574, U2 74HCT541

Commit message: move to Constant Register v2.0
Parts:
- removed D11: MB0, LED_SMD:LED_1206_3216Metric, symbol Device:LED_Small_ALT
- removed D12: MB1, LED_SMD:LED_1206_3216Metric, symbol Device:LED_Small_ALT
- removed D13: MB2, LED_SMD:LED_1206_3216Metric, symbol Device:LED_Small_ALT
- removed D14: MB3, LED_SMD:LED_1206_3216Metric, symbol Device:LED_Small_ALT
- removed D15: MB4, LED_SMD:LED_1206_3216Metric, symbol Device:LED_Small_ALT
- removed D16: MB5, LED_SMD:LED_1206_3216Metric, symbol Device:LED_Small_ALT
- removed D17: MB6, LED_SMD:LED_1206_3216Metric, symbol Device:LED_Small_ALT
- removed D18: MB7, LED_SMD:LED_1206_3216Metric, symbol Device:LED_Small_ALT
- removed RN4, RN5: R_Pack04, Resistor_SMD:R_Array_Convex_4x1206, symbol Device:R_Pack04
- removed U2: 74HCT541, Package_SO:SOIC-20W_7.5x12.8mm_P1.27mm, symbol 74xx:74HCT541
- added C4: C, Capacitor_SMD:C_1206_3216Metric, symbol Device:C
- added U2: 74HCT574, Package_SO:SOIC-20W_7.5x12.8mm_P1.27mm, symbol 74xx:74HCT574
- added U3: 74HCT00, Package_SO:SOIC-14_3.9x8.7mm_P1.27mm, symbol 74xx:74HCT00
Connections:
- net A_Main: now also U2.1 (OE), U3.13, U3.9
- net GND: now also C4.2, U2.10 (GND), U3.7 (GND); no longer U1.1 (OE)
- net Load: now also U2.11 (Cp), U3.1
- net MB0: now also U2.19 (Q0)
- net MB1: now also U2.18 (Q1)
- net MB2: now also U2.17 (Q2)
- net MB3: now also U2.16 (Q3)
- net MB4: now also U2.15 (Q4)
- net MB5: now also U2.14 (Q5)
- net MB6: now also U2.13 (Q6)
- net MB7: now also U2.12 (Q7)
- net MD0: now also U2.2 (D0)
- net MD1: now also U2.3 (D1)
- net MD2: now also U2.4 (D2)
- net MD3: now also U2.5 (D3)
- net MD4: now also U2.6 (D4)
- net MD5: now also U2.7 (D5)
- net MD6: now also U2.8 (D6)
- net MD7: now also U2.9 (D7)
- net VCC: now also C4.1, U2.20 (VCC), U3.14 (VCC)
- new net: U3.4, U3.5, U3.8
- new net: U3.10, U3.11, U3.2
- new net: U3.12, U3.3
- new net Reg_Valid: U1.1 (OE), U3.6
Other:
- title: Constants Register -> Constants Register v2.0
- moved on the sheet: D10, D9
